File: cad/motor/hbridge.kicad_sch (KiCad schematic)
At the start: 12 parts, among them Q1 NMOS, Q2 NMOS, Q3 PMOS, Q4 PMOS, Q5 NMOS, Q7 PMOS, Q8 PMOS

Commit message: enable/disable
Parts:
- added Q15: NMOS, symbol Simulation_SPICE:NMOS
- added Q17, Q19, Q21: PMOS, symbol Simulation_SPICE:PMOS
- added R1, R3: 1k, symbol Device:R
- added R15, R19, R21: 100, symbol Device:R
Connections:
- net GATE_1: now also R19.1; no longer Q2.2 (G), R5.1
- net GATE_2: now also R21.1; no longer Q1.2 (G), R2.1
- net GND: now also Q15.3 (S), R1.2
- net VDD: now also Q21.1 (D), R3.1; no longer Q7.3 (S), Q8.3 (S)
- net VBB renamed DIR
- new net: Q21.3 (S), Q7.3 (S), Q8.3 (S)
- new net: Q19.3 (S), R19.2
- new net: Q17.3 (S), R21.2
- new net: Q15.1 (D), R15.2, R3.2
- new net: Q17.2 (G), Q19.2 (G), Q21.2 (G), R15.1
- new net DISABLE: Q15.2 (G), R1.1
- new net GATE_3: Q19.1 (D), Q2.2 (G), R5.1
- new net GATE_4: Q1.2 (G), Q17.1 (D), R2.1
Other:
- moved on the sheet: Q1, Q2, Q3, Q4, Q5, Q7, Q8, R11, R4
