File: cad/kicad/galvo.kicad_sch (KiCad schematic)
At the start: 23 parts, among them Q1 NPN, Q10 NMOS, Q2 PMOS, Q3 NMOS, Q4 NMOS, Q5 NMOS, Q6 NPN, Q7 NMOS, Q8 NMOS, Q9 PMOS

Commit message: save and quit
Parts:
- removed L2: 30uH, symbol Device:L
- removed Q1: NPN, symbol Simulation_SPICE:NPN
- removed Q10, Q3, Q4, Q8: NMOS, symbol Simulation_SPICE:NMOS
- removed Q2, Q9: PMOS, symbol Simulation_SPICE:PMOS
- added Q1, Q10, Q13, Q16: PNP, symbol Simulation_SPICE:PNP
- added Q11, Q12, Q14, Q15, Q2, Q3, Q9: NPN, symbol Simulation_SPICE:NPN
- added Q4, Q8: PMOS, symbol Simulation_SPICE:PMOS
- added R10, R13: 100, symbol Device:R
- added R11: 1k, symbol Device:R
- added R12, R9: 5k, symbol Device:R
- added V4, V5: VPULSE, symbol Simulation_SPICE:VPULSE
- L1: value 30uH -> 40uH
- R2, R7: value 1k -> 20
- R3: value 100 -> 2k
- R4: value 3 -> 8
- R6: value 3 -> 2k
- R8: value 100 -> 1k
- V2: value 12V -> 12v
Connections:
- net GND: now also Q1.1 (C), Q10.1 (C), Q11.3 (E), Q13.1 (C), Q14.3 (E), Q16.1 (C), Q3.3 (E), V4.2, V5.2
- net VGATE: now also R2.2, Q8.2 (G); no longer Q5.2 (G), R3.1
- net VGATE2: now also R7.2, Q4.2 (G); no longer Q7.2 (G), R8.1
- net rail: now reaches R6.1
- net rail: now also R3.1, V2.1, Q12.1 (C), Q15.1 (C), Q2.1 (C), Q4.3 (S), Q8.3 (S), Q9.1 (C), R12.1, R9.1
- net at R6.2: now also Q6.1 (C), Q10.2 (B), Q9.2 (B); no longer Q7.1 (D)
- net at R8.2: now also Q11.2 (B)
- net at R3.2: now also Q1.2 (B), Q2.2 (B), Q3.1 (C)
- net at R4.2: now also Q7.1 (D), Q4.1 (D); no longer Q5.1 (D)
- net at R1.2: now also Q3.2 (B)
- new net: R11.1, V5.1
- new net: Q12.3 (E), Q13.3 (E), R10.1
- new net: Q10.3 (E), Q9.3 (E), R7.1
- new net: Q1.3 (E), Q2.3 (E), R2.1
- new net: Q11.1 (C), Q12.2 (B), Q13.2 (B), R9.2
- new net: Q14.1 (C), Q15.2 (B), Q16.2 (B), R12.2
- new net: Q15.3 (E), Q16.3 (E), R13.1
- new net: L1.1, Q5.1 (D), Q8.1 (D)
- new net: R8.1, V4.1
- new net: Q14.2 (B), R11.2
- new net VGATE3: Q5.2 (G), R10.2
- new net VGATE4: Q7.2 (G), R13.2
- no-connect marks 2 -> 0
Other:
- moved on the sheet: L1, Q5, Q7, R1, R4
