File: cad/kicad/galvo2.kicad_sch (KiCad schematic)
At the start: 2 parts

Commit message: save and quit
Parts:
- removed L1: ${SIM.PARAMS}, symbol Device:L
- added I1: 30uA, symbol Simulation_SPICE:IDC
- added V1: 3.3V, symbol Simulation_SPICE:VDC
- R1: value 1 -> 100k
Connections:
- net GND: now reaches R1.2
- net GND: now also I1.1, V1.2
- net at R1.1: now also I1.2
Other:
- note removed: ".tran 1u 100u UIC"
